File: EtherDue.kicad_pcb (KiCad board)
At the start: 4 copper layers, 185 x 104 mm, 596 parts, among them IC201 ATSAM3X8E, IC301 ATMEGA16U2, IC601 W5100, P101 CONN_02X04, P102 MSTBV3, P103 MSTBV3, P104 MSTBV6, P1101 CONN_01X02, P1102 CONN_01X02, P1201 CONN_01X02, P1202 CONN_01X02, P1301 CONN_01X02, P1302 CONN_01X02, P1401 CONN_01X02, P1402 CONN_01X02, P301 USB_5PIN_SHELL, P401 USB_5PIN_SHELL, P801 MSTBV2, P901 677006144621, P902 677006144621, Q1001 BSS308, Q101 IPB020NE7N3G, Q102 IPB020NE7N3G, Q1501 BSS123, Q1502 BSS123, Q1601 BSS123, Q1602 BSS123, Q1701 BSS123, Q1702 BSS123, Q1703 BSS308, Q1704 BSS308, Q1801 BSS123, Q1802 BSS123, Q1803 BSS308, Q1804 BSS308, Q1901 BSS123, Q1902 BSS123, Q1903 BSS308, Q1904 BSS308, Q501 BC847BSMD, Q601 2N7002, SW1701 SW_PUSH, SW1801 SW_PUSH, SW1901 SW_PUSH, SW201 ERASE, SW202 RESET, U1001 AD7294BSUZ, U101 AD7415, U1101 ADL5513, U1102 REG101NA-5, U1201 ADL5513, U1202 REG101NA-5, U1301 ADL5513, U1302 REG101NA-5, U1401 ADL5513, U1402 REG101NA-5, U1501 4013_with_supply, U1701 MCP6H04, U1702 INA207, U1703 MEU1S1212ZC, U1801 INA207, U1802 MEU1S1212ZC, U1901 INA207, U1902 MEU1S1212ZC, U202 FDN340P, U203 LMV358IPWR, U501 POWERJACK, U502 LM2734Y, U503 FDN340P, U504 FDN340P, U505 NCP1117ST33T3G, U602 HY931147C, U603 APX811-31UG-7, U701 MICROSD, U702 24AA025E48, U801 TPS7A4501DCQT, U802 TPS7A4501DCQT, U803 TPS7A4501DCQT, U804 REG101NA-5, U901 TJA1040T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

Commit message: just before finishing DRC errors
Parts:
- D201, D202, D203, D204, D302, D303, D601, D602, D603, D604, D605, D606: footprint LEDs:LED-0603 -> zeilhofer:LED-0603
- JP601: footprint FT:FT-POE-MODULE-NOOUTLINE -> zeilhofer:FT-POE-MODULE-NOOUTLINE
Connections:
- R1501 pad 1: PWM2 -> PIN48
- R1601 pad 1: PWM3 -> PIN49
- U1501 pad 11: PIN23 -> PIN47
- U1501 pad 3: PIN22 -> PIN46
Routing:
- net SCK: track 37.3 -> 107.6 mm, vias 2 -> 5
- net GND: track 2496.8 -> 2427.9 mm, vias 431 -> 533
- net PIN22: track 94.4 -> 53.2 mm, vias 3 -> 1
- net PIN23: track 136.4 -> 97.1 mm, vias 10 -> 8
- net /Analog I/O/+3V3: track 316.1 -> 353.4 mm
- net PWM13: track 26.0 -> 56.9 mm, vias 0 -> 1
- net PIN47: track 53.4 -> 77.0 mm, vias 2 -> 4
- net PIN46: track 61.1 -> 84.3 mm, vias 1 -> 4
- net PIN41: track 51.4 -> 72.5 mm, vias 0 -> 1
- net PIN49: track 50.6 -> 69.3 mm, vias 1 -> 3
- net PIN48: track 70.7 -> 87.7 mm, vias 2 -> 4
- net (no net): track 18.1 -> 2.54 mm, vias 8 -> 4
- net Net-(Q1802-PadD): track 4.97 -> 14.6 mm, vias 0 -> 2
- net AD2: track 200.0 -> 190.4 mm
- net /PA-Monitor Power Supply/VIN: track 101.5 -> 110.8 mm, vias 2 -> 6
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Other:
- board text removed: "Alert-LED"
