File: EtherDue.kicad_pcb (KiCad board)
At the start: 4 copper layers, 185 x 104 mm, 596 parts, among them IC201 ATSAM3X8E, IC301 ATMEGA16U2, IC601 W5100, P101 CONN_02X04, P102 MSTBV3, P103 MSTBV3, P104 MSTBV6, P1101 CONN_01X02, P1102 CONN_01X02, P1201 CONN_01X02, P1202 CONN_01X02, P1301 CONN_01X02, P1302 CONN_01X02, P1401 CONN_01X02, P1402 CONN_01X02, P301 USB_5PIN_SHELL, P401 USB_5PIN_SHELL, P801 MSTBV2, P901 677006144621, P902 677006144621, Q1001 BSS308, Q101 IPB020NE7N3G, Q102 IPB020NE7N3G, Q1501 BSS123, Q1502 BSS123, Q1601 BSS123, Q1602 BSS123, Q1701 BSS123, Q1702 BSS123, Q1703 BSS308, Q1704 BSS308, Q1801 BSS123, Q1802 BSS123, Q1803 BSS308, Q1804 BSS308, Q1901 BSS123, Q1902 BSS123, Q1903 BSS308, Q1904 BSS308, Q501 BC847BSMD, Q601 2N7002, SW1701 SW_PUSH, SW1801 SW_PUSH, SW1901 SW_PUSH, SW201 ERASE, SW202 RESET, U1001 AD7294BSUZ, U101 AD7415, U1101 ADL5513, U1102 REG101NA-5, U1201 ADL5513, U1202 REG101NA-5, U1301 ADL5513, U1302 REG101NA-5, U1401 ADL5513, U1402 REG101NA-5, U1501 4013_with_supply, U1701 MCP6H04, U1702 INA207, U1703 MEU1S1212ZC, U1801 INA207, U1802 MEU1S1212ZC, U1901 INA207, U1902 MEU1S1212ZC, U202 FDN340P, U203 LMV358IPWR, U501 POWERJACK, U502 LM2734Y, U503 FDN340P, U504 FDN340P, U505 NCP1117ST33T3G, U602 HY931147C, U603 APX811-31UG-7, U701 MICROSD, U702 24AA025E48, U801 TPS7A4501DCQT, U802 TPS7A4501DCQT, U803 TPS7A4501DCQT, U804 REG101NA-5, U901 TJA1040T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

Commit message: Updates im Zuge des Tutorials
Parts:
- added C209: 10nF, FT:C0402, F.Cu at (66.4, 244.9)
- added C210: 10uF, FT:SM0603_Capa, F.Cu at (63.9, 244.6)
- added C404: 22pF, FT:C0402, F.Cu at (87.1, 225.5)
- added C405: 22pF, FT:C0402, F.Cu at (86.4, 231.4)
- added C406: 22pF, FT:C0402, F.Cu at (83.4, 231.4)
- added C407: 22pF, FT:C0402, F.Cu at (84.9, 231.4)
- added R209: 33R, Resistors_SMD:R_0402, F.Cu at (71.2, 235.3)
- C1105, C1107, C1205, C1207, C1305, C1307, C1405, C1407: footprint Capacitors_SMD:C_0402 -> Capacitors_SMD:C_0603
- C1110, C1210, C1310, C1410: value 47p/X7R -> 47p/C0G
- P901, P902: footprint eagle-InputOutputIO:677006144621 -> zeilhofer:Firewire-Female-WE677006144621
- moved C1105 134.5 mm to (127.9, 288.6), turned to 0 degrees
- moved C1107 128.0 mm to (135.6, 288.6), turned to 0 degrees
- moved C1205 124.5 mm to (127.9, 300.3), turned to 0 degrees
- moved C1207 117.5 mm to (135.6, 300.3), turned to 0 degrees
- moved C1305 86.0 mm to (146.4, 288.6), turned to 0 degrees
- moved C1405 78.3 mm to (146.4, 300.3), turned to 0 degrees
- moved C1307 78.0 mm to (154.0, 288.6), turned to 0 degrees
- moved C1407 69.4 mm to (154.0, 300.3), turned to 0 degrees
- moved P902 11.4 mm to (139.5, 264.3)
- moved P901 11.4 mm to (150.9, 264.3)
- moved C518 2.18 mm to (61.5, 244.3)
- moved L504 0.89 mm to (62.7, 242.4)
- moved C204 0.73 mm to (61.2, 245.7)
Connections:
- IC201 pad 35: Net-(C201-Pad2) -> Net-(IC201-Pad35)
Routing:
- net /PA-Monitor Power Supply/VIN: track 110.8 -> 135.1 mm
- net GND: track 2467.2 -> 2476.3 mm, vias 547 -> 549
- net Net-(C201-Pad2): track 15.8 -> 11.6 mm
- net Net-(IC201-Pad35): track 0.00 -> 3.43 mm
- net +3.3V: track 157.5 -> 160.8 mm, vias 26 -> 27
- net JTAG_TCK: track 34.5 -> 36.9 mm
- net JTAG_TDO: track 14.9 -> 17.1 mm
- net /Analog I/O/+12V: track 120.6 -> 122.5 mm
- net RXD0: track 39.9 -> 38.4 mm
- net /Connectors//MASTER-RESET: track 104.1 -> 102.7 mm
- net JTAG_TMS: track 41.0 -> 42.2 mm
- net PWM2: track 42.5 -> 41.4 mm
- net /CAN-Bus/+5V: track 48.9 -> 47.8 mm, vias 1 -> 0
- net /MCU/VDDOUTMI: track 7.45 -> 8.44 mm
- net JTAG_TDI: track 36.9 -> 37.9 mm
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- removed copper zone on Inner.VCC, net /Analog I/O/+12V
- removed copper zone on Inner.VCC, net /CAN-Bus/+5V
- removed copper zone on Inner.VCC, net /PA-Monitor Power Supply/VIN
