File: EtherDue.sch (KiCad schematic (older format))
At the start: 27 parts, among them P101 CONN_02X04, P102 MSTBV3, P103 MSTBV3, P104 MSTBV6, Q101 IPB020NE7N3G, Q102 IPB020NE7N3G, U101 AD7415, U1701 MCP6H04

Commit message: just before finishing DRC errors
Changed lines of the file:
@@
 AD5
 Text GLabel 9600 3600 0    60   Input ~ 0
-PWM2
+PIN48
 Text GLabel 9600 5150 0    60   Input ~ 0
-PWM3
+PIN49
 Text GLabel 9600 3700 0    60   Input ~ 0
-PIN22
+PIN46
 Text GLabel 9600 5250 0    60   Input ~ 0
-PIN23
+PIN47
 Text GLabel 3450 11000 2    60   Output ~ 0
 PIN24
