File: EtherDue_Mega16U2.sch (KiCad schematic (older format))
At the start: 25 parts, among them IC301 ATMEGA16U2, P301 USB_5PIN_SHELL, X301 TXC 7A 16MHz 18pF

Commit message: exported cmp-file from PCB and back imported it into the schematic. then exported BOM with kicad2csvbom tool
Parts:
- C301, C302, C303, C304, C305: footprint SMD_Packages:SMD-0402_c -> SM0402
- D302, D303: footprint LEDs:LED-0603 -> zeilhofer:LED-0603
- F301: footprint SMD_Packages:SMD-1812 -> SM1812
- R301, R302, R303, R304, R305, R306, R307, R308, R309, R310: footprint SMD_Packages:SMD-0402_r -> SM0402_r
Changed lines of the file:
@@
 F 0 "R305" V 9730 5550 50  0000 C CNN
 F 1 "2K7" V 9650 5550 50  0000 C CNN
-F 2 "SMD_Packages:SMD-0402_r" H 9650 5550 60  0001 C CNN
+F 2 "SM0402_r" H 9650 5550 60  0001 C CNN
 F 3 "" H 9650 5550 60  0001 C CNN
 	1    9650 5550
@@
 F 0 "R304" V 9330 5300 50  0000 C CNN
 F 1 "1K5" V 9250 5300 50  0000 C CNN
-F 2 "SMD_Packages:SMD-0402_r" H 9250 5300 60  0001 C CNN
+F 2 "SM0402_r" H 9250 5300 60  0001 C CNN
 F 3 "" H 9250 5300 60  0001 C CNN
 	1    9250 5300
@@
 F 0 "R308" V 10080 4200 50  0000 C CNN
 F 1 "1K" V 10000 4200 50  0000 C CNN
-F 2 "SMD_Packages:SMD-0402_r" H 10000 4200 60  0001 C CNN
+F 2 "SM0402_r" H 10000 4200 60  0001 C CNN
 F 3 "" H 10000 4200 60  0001 C CNN
 	1    10000 4200
@@
 F 0 "R309" V 10080 4500 50  0000 C CNN
 F 1 "1K" V 10000 4500 50  0000 C CNN
-F 2 "SMD_Packages:SMD-0402_r" H 10000 4500 60  0001 C CNN
+F 2 "SM0402_r" H 10000 4500 60  0001 C CNN
 F 3 "" H 10000 4500 60  0001 C CNN
 	1    10000 4500
@@
 F 0 "D303" H 9300 4600 50  0000 C CNN
 F 1 "YELLOW" H 9300 4400 50  0000 C CNN
-F 2 "LEDs:LED-0603" H 9300 4500 60  0001 C CNN
+F 2 "zeilhofer:LED-0603" H 9300 4500 60  0001 C CNN
 F 3 "" H 9300 4500 60  0001 C CNN
 	1    9300 4500
@@
 F 0 "D302" H 9300 4300 50  0000 C CNN
 F 1 "YELLOW" H 9300 4100 50  0000 C CNN
-F 2 "LEDs:LED-0603" H 9300 4200 60  0001 C CNN
+F 2 "zeilhofer:LED-0603" H 9300 4200 60  0001 C CNN
 F 3 "" H 9300 4200 60  0001 C CNN
 	1    9300 4200
@@
 F 0 "R310" V 11080 4450 50  0000 C CNN
 F 1 "10K" V 11000 4450 50  0000 C CNN
-F 2 "SMD_Packages:SMD-0402_r" H 11000 4450 60  0001 C CNN
+F 2 "SM0402_r" H 11000 4450 60  0001 C CNN
 F 3 "" H 11000 4450 60  0001 C CNN
 	1    11000 4450
@@
 F 0 "R307" V 10080 3550 50  0000 C CNN
 F 1 "1K" V 10000 3550 50  0000 C CNN
-F 2 "SMD_Packages:SMD-0402_r" H 10000 3550 60  0001 C CNN
+F 2 "SM0402_r" H 10000 3550 60  0001 C CNN
 F 3 "" H 10000 3550 60  0001 C CNN
 	1    10000 3550
@@
 F 0 "R306" V 10080 2500 50  0000 C CNN
 F 1 "1K" V 10000 2500 50  0000 C CNN
-F 2 "SMD_Packages:SMD-0402_r" H 10000 2500 60  0001 C CNN
+F 2 "SM0402_r" H 10000 2500 60  0001 C CNN
 F 3 "" H 10000 2500 60  0001 C CNN
 	1    10000 2500
@@
 F 0 "R302" V 2930 4450 50  0000 C CNN
 F 1 "22R" V 2850 4450 50  0000 C CNN
-F 2 "SMD_Packages:SMD-0402_r" H 2850 4450 60  0001 C CNN
+F 2 "SM0402_r" H 2850 4450 60  0001 C CNN
 F 3 "" H 2850 4450 60  0001 C CNN
 	1    2850 4450
@@
 F 0 "R301" V 2930 4250 50  0000 C CNN
 F 1 "22R" V 2850 4250 50  0000 C CNN
-F 2 "SMD_Packages:SMD-0402_r" H 2850 4250 60  0001 C CNN
+F 2 "SM0402_r" H 2850 4250 60  0001 C CNN
 F 3 "" H 2850 4250 60  0001 C CNN
 	1    2850 4250
@@
 F 0 "C301" H 2500 3850 50  0000 L CNN
 F 1 "100nF" H 2500 3650 50  0000 L CNN
-F 2 "SMD_Packages:SMD-0402_c" H 2450 3750 60  0001 C CNN
+F 2 "SM0402" H 2450 3750 60  0001 C CNN
 F 3 "" H 2450 3750 60  0001 C CNN
 	1    2450 3750
@@
 F 0 "F301" H 2100 3550 40  0000 C CNN
 F 1 "500mA PTC 1812" H 2000 3350 40  0000 C CNN
-F 2 "SMD_Packages:SMD-1812" H 2000 3500 60  0001 C CNN
+F 2 "SM1812" H 2000 3500 60  0001 C CNN
 F 3 "" H 2000 3500 60  0001 C CNN
 	1    2000 3500
@@
 F 0 "C305" H 4550 4600 50  0000 L CNN
 F 1 "1uF" H 4550 4400 50  0000 L CNN
-F 2 "SMD_Packages:SMD-0402_c" H 4500 4500 60  0001 C CNN
+F 2 "SM0402" H 4500 4500 60  0001 C CNN
 F 3 "" H 4500 4500 60  0001 C CNN
 	1    4500 4500
@@
 F 0 "C302" H 4150 4600 50  0000 L CNN
 F 1 "100nF" H 4150 4400 50  0000 L CNN
-F 2 "SMD_Packages:SMD-0402_c" H 4100 4500 60  0001 C CNN
+F 2 "SM0402" H 4100 4500 60  0001 C CNN
 F 3 "" H 4100 4500 60  0001 C CNN
 	1    4100 4500
@@
 F 0 "C304" H 4400 3250 50  0000 L CNN
 F 1 "22pF" H 4400 3050 50  0000 L CNN
-F 2 "SMD_Packages:SMD-0402_c" H 4350 3150 60  0001 C CNN
+F 2 "SM0402" H 4350 3150 60  0001 C CNN
 F 3 "" H 4350 3150 60  0001 C CNN
 	1    4350 3150
@@
 F 0 "C303" H 4400 2850 50  0000 L CNN
 F 1 "22pF" H 4400 2650 50  0000 L CNN
-F 2 "SMD_Packages:SMD-0402_c" H 4350 2750 60  0001 C CNN
+F 2 "SM0402" H 4350 2750 60  0001 C CNN
 F 3 "" H 4350 2750 60  0001 C CNN
 	1    4350 2750
@@
 F 0 "R303" V 5180 2000 50  0000 C CNN
 F 1 "10K" V 5100 2000 50  0000 C CNN
-F 2 "SMD_Packages:SMD-0402_r" H 5100 2000 60  0001 C CNN
+F 2 "SM0402_r" H 5100 2000 60  0001 C CNN
 F 3 "" H 5100 2000 60  0001 C CNN
 	1    5100 2000
