File: EtherDue_Ethernet.sch (KiCad schematic (older format))
At the start: 33 parts, among them IC601 W5100, Q601 2N7002, U602 HY931147C, U603 APX811-31UG-7, X601 TXC 7A 25MHz 18pF

Commit message: exported cmp-file from PCB and back imported it into the schematic. then exported BOM with kicad2csvbom tool
Parts:
- C601, C602, C603, C605, C607, C609, C610, C611: footprint SMD_Packages:SMD-0402_c -> SM0402
- D601, D602, D603, D604, D605, D606: footprint LEDs:LED-0603 -> zeilhofer:LED-0603
- JP601: footprint FT:FT-POE-MODULE-NOOUTLINE -> zeilhofer:FT-POE-MODULE-NOOUTLINE
- R602, R603, R606, R607: footprint SMD_Packages:SMD-0402_r -> SM0402_r
Changed lines of the file:
@@
 F 0 "C609" H 6700 4650 50  0000 L CNN
 F 1 "100nF" H 6700 4450 50  0000 L CNN
-F 2 "SMD_Packages:SMD-0402_c" H 6650 4550 60  0001 C CNN
+F 2 "SM0402" H 6650 4550 60  0001 C CNN
 F 3 "" H 6650 4550 60  0001 C CNN
 	1    6650 4550
@@
 F 0 "C610" H 7000 4650 50  0000 L CNN
 F 1 "100nF" H 7000 4450 50  0000 L CNN
-F 2 "SMD_Packages:SMD-0402_c" H 6950 4550 60  0001 C CNN
+F 2 "SM0402" H 6950 4550 60  0001 C CNN
 F 3 "" H 6950 4550 60  0001 C CNN
 	1    6950 4550
@@
 F 0 "JP601" H 500 7200 50  0000 C CNN
 F 1 "M04" H 500 6700 40  0000 C CNN
-F 2 "FT:FT-POE-MODULE-NOOUTLINE" H 600 7100 60  0001 C CNN
+F 2 "zeilhofer:FT-POE-MODULE-NOOUTLINE" H 600 7100 60  0001 C CNN
 F 3 "" H 600 7100 60  0001 C CNN
 	1    600  7100
@@
 F 0 "C611" H 7300 4050 50  0000 L CNN
 F 1 "100nF" H 7300 3850 50  0000 L CNN
-F 2 "SMD_Packages:SMD-0402_c" H 7250 3950 60  0001 C CNN
+F 2 "SM0402" H 7250 3950 60  0001 C CNN
 F 3 "" H 7250 3950 60  0001 C CNN
 	1    7250 3950
@@
 F 0 "C603" H 2800 1500 50  0000 L CNN
 F 1 "100nF" H 2800 1300 50  0000 L CNN
-F 2 "SMD_Packages:SMD-0402_c" H 2750 1400 60  0001 C CNN
+F 2 "SM0402" H 2750 1400 60  0001 C CNN
 F 3 "" H 2750 1400 60  0001 C CNN
 	1    2750 1400
@@
 F 0 "C605" H 4100 1450 50  0000 L CNN
 F 1 "100nF" H 4100 1250 50  0000 L CNN
-F 2 "SMD_Packages:SMD-0402_c" H 4050 1350 60  0001 C CNN
+F 2 "SM0402" H 4050 1350 60  0001 C CNN
 F 3 "" H 4050 1350 60  0001 C CNN
 	1    4050 1350
@@
 F 0 "C607" H 4450 1450 50  0000 L CNN
 F 1 "100nF" H 4450 1250 50  0000 L CNN
-F 2 "SMD_Packages:SMD-0402_c" H 4400 1350 60  0001 C CNN
+F 2 "SM0402" H 4400 1350 60  0001 C CNN
 F 3 "" H 4400 1350 60  0001 C CNN
 	1    4400 1350
@@
 F 0 "D604" H 7650 1950 50  0000 C CNN
 F 1 "RED" H 7400 1950 50  0000 C CNN
-F 2 "LEDs:LED-0603" H 7500 2050 60  0001 C CNN
+F 2 "zeilhofer:LED-0603" H 7500 2050 60  0001 C CNN
 F 3 "" H 7500 2050 60  0001 C CNN
 	1    7500 2050
@@
 F 0 "D605" H 7650 2150 50  0000 C CNN
 F 1 "YELLOW" H 7350 2150 50  0000 C CNN
-F 2 "LEDs:LED-0603" H 7500 2250 60  0001 C CNN
+F 2 "zeilhofer:LED-0603" H 7500 2250 60  0001 C CNN
 F 3 "" H 7500 2250 60  0001 C CNN
 	1    7500 2250
@@
 F 0 "D606" H 7650 2350 50  0000 C CNN
 F 1 "YELLOW" H 7400 2350 50  0000 C CNN
-F 2 "LEDs:LED-0603" H 7500 2450 60  0001 C CNN
+F 2 "zeilhofer:LED-0603" H 7500 2450 60  0001 C CNN
 F 3 "" H 7500 2450 60  0001 C CNN
 	1    7500 2450
@@
 F 0 "D603" H 7650 1700 50  0000 C CNN
 F 1 "GREEN" H 7350 1700 50  0000 C CNN
-F 2 "LEDs:LED-0603" H 7500 1800 60  0001 C CNN
+F 2 "zeilhofer:LED-0603" H 7500 1800 60  0001 C CNN
 F 3 "" H 7500 1800 60  0001 C CNN
 	1    7500 1800
@@
 F 0 "D602" H 7650 1500 50  0000 C CNN
 F 1 "GREEN" H 7350 1500 50  0000 C CNN
-F 2 "LEDs:LED-0603" H 7500 1600 60  0001 C CNN
+F 2 "zeilhofer:LED-0603" H 7500 1600 60  0001 C CNN
 F 3 "" H 7500 1600 60  0001 C CNN
 	1    7500 1600
@@
 F 0 "D601" H 7650 1250 50  0000 C CNN
 F 1 "YELLOW" H 7350 1250 50  0000 C CNN
-F 2 "LEDs:LED-0603" H 7500 1350 60  0001 C CNN
+F 2 "zeilhofer:LED-0603" H 7500 1350 60  0001 C CNN
 F 3 "" H 7500 1350 60  0001 C CNN
 	1    7500 1350
@@
 F 0 "C602" H 1400 1950 50  0000 L CNN
 F 1 "22pF" H 1400 1750 50  0000 L CNN
-F 2 "SMD_Packages:SMD-0402_c" H 1350 1850 60  0001 C CNN
+F 2 "SM0402" H 1350 1850 60  0001 C CNN
 F 3 "" H 1350 1850 60  0001 C CNN
 	1    1350 1850
@@
 F 0 "C601" H 1050 2700 50  0000 L CNN
 F 1 "22pF" H 1050 2500 50  0000 L CNN
-F 2 "SMD_Packages:SMD-0402_c" H 1000 2600 60  0001 C CNN
+F 2 "SM0402" H 1000 2600 60  0001 C CNN
 F 3 "" H 1000 2600 60  0001 C CNN
 	1    1000 2600
@@
 F 0 "R602" V 1830 1900 50  0000 C CNN
 F 1 "1M" V 1750 1900 50  0000 C CNN
-F 2 "SMD_Packages:SMD-0402_r" H 1750 1900 60  0001 C CNN
+F 2 "SM0402_r" H 1750 1900 60  0001 C CNN
 F 3 "" H 1750 1900 60  0001 C CNN
 	1    1750 1900
@@
 F 0 "R603" V 6280 3650 50  0000 C CNN
 F 1 "12K3 1%" V 6100 3650 50  0000 C CNN
-F 2 "SMD_Packages:SMD-0402_r" H 6200 3650 60  0001 C CNN
+F 2 "SM0402_r" H 6200 3650 60  0001 C CNN
 F 3 "" H 6200 3650 60  0001 C CNN
 	1    6200 3650
@@
 F 0 "R606" V 8280 4300 40  0000 C CNN
 F 1 "1K" V 8207 4301 40  0000 C CNN
-F 2 "SMD_Packages:SMD-0402_r" V 8130 4300 30  0000 C CNN
+F 2 "SM0402_r" V 8130 4300 30  0000 C CNN
 F 3 "~" H 8200 4300 30  0000 C CNN
 	1    8200 4300
@@
 F 0 "R607" V 8280 4600 40  0000 C CNN
 F 1 "1K" V 8207 4601 40  0000 C CNN
-F 2 "SMD_Packages:SMD-0402_r" V 8130 4600 30  0000 C CNN
+F 2 "SM0402_r" V 8130 4600 30  0000 C CNN
 F 3 "~" H 8200 4600 30  0000 C CNN
 	1    8200 4600
