File: EtherDue_Power.sch (KiCad schematic (older format))
At the start: 47 parts, among them Q501 BC847BSMD, U203 LMV358IPWR, U501 POWERJACK, U502 LM2734Y, U503 FDN340P, U504 FDN340P, U505 NCP1117ST33T3G

Commit message: exported cmp-file from PCB and back imported it into the schematic. then exported BOM with kicad2csvbom tool
Parts:
- C502: footprint SMD_Packages:SMD-1206 -> SM1206
- C503, C504, C505, C509, C511, C512, C513, C514, C515, C516, C520, C521, C522, C523, C524, C526, C527: footprint SMD_Packages:SMD-0402_c -> SM0402
- R501, R503, R504, R505: footprint SMD_Packages:SMD-0402_r -> SM0402_r
Changed lines of the file:
@@
 F 0 "C514" H 9000 4800 50  0000 L CNN
 F 1 "100nF" H 9000 4600 50  0000 L CNN
-F 2 "SMD_Packages:SMD-0402_c" H 8950 4700 60  0001 C CNN
+F 2 "SM0402" H 8950 4700 60  0001 C CNN
 F 3 "" H 8950 4700 60  0001 C CNN
 	1    8950 4700
@@
 F 0 "C509" H 8150 4800 50  0000 L CNN
 F 1 "100nF" H 8150 4600 50  0000 L CNN
-F 2 "SMD_Packages:SMD-0402_c" H 8100 4700 60  0001 C CNN
+F 2 "SM0402" H 8100 4700 60  0001 C CNN
 F 3 "" H 8100 4700 60  0001 C CNN
 	1    8100 4700
@@
 F 0 "C516" H 8800 6250 50  0000 L CNN
 F 1 "100nF" H 8800 6050 50  0000 L CNN
-F 2 "SMD_Packages:SMD-0402_c" H 8750 6150 60  0001 C CNN
+F 2 "SM0402" H 8750 6150 60  0001 C CNN
 F 3 "" H 8750 6150 60  0001 C CNN
 	1    8750 6150
@@
 F 0 "C511" H 8500 6250 50  0000 L CNN
 F 1 "100nF" H 8500 6050 50  0000 L CNN
-F 2 "SMD_Packages:SMD-0402_c" H 8450 6150 60  0001 C CNN
+F 2 "SM0402" H 8450 6150 60  0001 C CNN
 F 3 "" H 8450 6150 60  0001 C CNN
 	1    8450 6150
@@
 F 0 "C521" H 9100 6250 50  0000 L CNN
 F 1 "100nF" H 9100 6050 50  0000 L CNN
-F 2 "SMD_Packages:SMD-0402_c" H 9050 6150 60  0001 C CNN
+F 2 "SM0402" H 9050 6150 60  0001 C CNN
 F 3 "" H 9050 6150 60  0001 C CNN
 	1    9050 6150
@@
 F 0 "C523" H 9450 6250 50  0000 L CNN
 F 1 "100nF" H 9450 6050 50  0000 L CNN
-F 2 "SMD_Packages:SMD-0402_c" H 9400 6150 60  0001 C CNN
+F 2 "SM0402" H 9400 6150 60  0001 C CNN
 F 3 "" H 9400 6150 60  0001 C CNN
 	1    9400 6150
@@
 F 0 "C526" H 10200 5600 50  0000 L CNN
 F 1 "100nF" H 10200 5400 50  0000 L CNN
-F 2 "SMD_Packages:SMD-0402_c" H 10150 5500 60  0001 C CNN
+F 2 "SM0402" H 10150 5500 60  0001 C CNN
 F 3 "" H 10150 5500 60  0001 C CNN
 	1    10150 5500
@@
 F 0 "C527" H 10550 5600 50  0000 L CNN
 F 1 "100nF" H 10550 5400 50  0000 L CNN
-F 2 "SMD_Packages:SMD-0402_c" H 10500 5500 60  0001 C CNN
+F 2 "SM0402" H 10500 5500 60  0001 C CNN
 F 3 "" H 10500 5500 60  0001 C CNN
 	1    10500 5500
@@
 F 0 "C524" H 9850 5600 50  0000 L CNN
 F 1 "100nF" H 9850 5400 50  0000 L CNN
-F 2 "SMD_Packages:SMD-0402_c" H 9800 5500 60  0001 C CNN
+F 2 "SM0402" H 9800 5500 60  0001 C CNN
 F 3 "" H 9800 5500 60  0001 C CNN
 	1    9800 5500
@@
 F 0 "C522" H 9500 5600 50  0000 L CNN
 F 1 "100nF" H 9500 5400 50  0000 L CNN
-F 2 "SMD_Packages:SMD-0402_c" H 9450 5500 60  0001 C CNN
+F 2 "SM0402" H 9450 5500 60  0001 C CNN
 F 3 "" H 9450 5500 60  0001 C CNN
 	1    9450 5500
@@
 F 0 "C515" H 8800 5600 50  0000 L CNN
 F 1 "100nF" H 8800 5400 50  0000 L CNN
-F 2 "SMD_Packages:SMD-0402_c" H 8750 5500 60  0001 C CNN
+F 2 "SM0402" H 8750 5500 60  0001 C CNN
 F 3 "" H 8750 5500 60  0001 C CNN
 	1    8750 5500
@@
 F 0 "C520" H 9150 5600 50  0000 L CNN
 F 1 "100nF" H 9150 5400 50  0000 L CNN
-F 2 "SMD_Packages:SMD-0402_c" H 9100 5500 60  0001 C CNN
+F 2 "SM0402" H 9100 5500 60  0001 C CNN
 F 3 "" H 9100 5500 60  0001 C CNN
 	1    9100 5500
@@
 F 0 "C513" H 8450 4150 50  0000 L CNN
 F 1 "100nF" H 8450 3950 50  0000 L CNN
-F 2 "SMD_Packages:SMD-0402_c" H 8400 4050 60  0001 C CNN
+F 2 "SM0402" H 8400 4050 60  0001 C CNN
 F 3 "" H 8400 4050 60  0001 C CNN
 	1    8400 4050
@@
 F 0 "C512" H 8450 3300 50  0000 L CNN
 F 1 "100nF" H 8450 3100 50  0000 L CNN
-F 2 "SMD_Packages:SMD-0402_c" H 8400 3200 60  0001 C CNN
+F 2 "SM0402" H 8400 3200 60  0001 C CNN
 F 3 "" H 8400 3200 60  0001 C CNN
 	1    8400 3200
@@
 F 0 "C504" H 4950 5300 50  0000 L CNN
 F 1 "100nF" H 4800 5100 50  0000 L CNN
-F 2 "SMD_Packages:SMD-0402_c" H 5050 5200 60  0001 C CNN
+F 2 "SM0402" H 5050 5200 60  0001 C CNN
 F 3 "" H 5050 5200 60  0001 C CNN
 	1    5050 5200
@@
 F 0 "C503" H 4600 5650 50  0000 L CNN
 F 1 "100nF" H 4600 5450 50  0000 L CNN
-F 2 "SMD_Packages:SMD-0402_c" H 4550 5550 60  0001 C CNN
+F 2 "SM0402" H 4550 5550 60  0001 C CNN
 F 3 "" H 4550 5550 60  0001 C CNN
 	1    4550 5550
@@
 F 0 "R501" V 2330 5350 50  0000 C CNN
 F 1 "1K" V 2250 5350 50  0000 C CNN
-F 2 "SMD_Packages:SMD-0402_r" H 2250 5350 60  0001 C CNN
+F 2 "SM0402_r" H 2250 5350 60  0001 C CNN
 F 3 "" H 2250 5350 60  0001 C CNN
 	1    2250 5350
@@
 F 0 "R505" V 6330 3000 50  0000 C CNN
 F 1 "10K" V 6250 3000 50  0000 C CNN
-F 2 "SMD_Packages:SMD-0402_r" H 6250 3000 60  0001 C CNN
+F 2 "SM0402_r" H 6250 3000 60  0001 C CNN
 F 3 "" H 6250 3000 60  0001 C CNN
 	1    6250 3000
@@
 F 0 "R504" V 6330 2350 50  0000 C CNN
 F 1 "52K3" V 6250 2350 50  0000 C CNN
-F 2 "SMD_Packages:SMD-0402_r" H 6250 2350 60  0001 C CNN
+F 2 "SM0402_r" H 6250 2350 60  0001 C CNN
 F 3 "" H 6250 2350 60  0001 C CNN
 	1    6250 2350
@@
 F 0 "C505" H 6150 1550 50  0000 L CNN
 F 1 "10nF" H 6150 1350 50  0000 L CNN
-F 2 "SMD_Packages:SMD-0402_c" H 6100 1450 60  0001 C CNN
+F 2 "SM0402" H 6100 1450 60  0001 C CNN
 F 3 "" H 6100 1450 60  0001 C CNN
 	1    6100 1450
@@
 F 0 "R503" V 4230 1650 50  0000 C CNN
 F 1 "10K" V 4150 1650 50  0000 C CNN
-F 2 "SMD_Packages:SMD-0402_r" H 4150 1650 60  0001 C CNN
+F 2 "SM0402_r" H 4150 1650 60  0001 C CNN
 F 3 "" H 4150 1650 60  0001 C CNN
 	1    4150 1650
@@
 F 0 "C502" V 3300 1500 50  0000 L CNN
 F 1 "10uF 25V" V 3600 1400 50  0000 L CNN
-F 2 "SMD_Packages:SMD-1206" H 3450 1600 60  0001 C CNN
+F 2 "SM1206" H 3450 1600 60  0001 C CNN
 F 3 "" H 3450 1600 60  0001 C CNN
 	1    3450 1600
