File: EtherDue_peripherals.sch (KiCad schematic (older format))
At the start: 5 parts, among them U701 MICROSD, U702 24AA025E48

Commit message: exported cmp-file from PCB and back imported it into the schematic. then exported BOM with kicad2csvbom tool
Parts:
- C701: footprint SMD_Packages:SMD-0402_c -> SM0402
Changed lines of the file:
@@
 F 0 "C701" H 1400 2000 40  0000 L CNN
 F 1 "100nF" H 1406 1815 40  0000 L CNN
-F 2 "SMD_Packages:SMD-0402_c" H 1438 1750 30  0000 C CNN
+F 2 "SM0402" H 1438 1750 30  0000 C CNN
 F 3 "~" H 1400 1900 60  0000 C CNN
 	1    1400 1900
