File: can-bus.sch (KiCad schematic (older format))
At the start: 15 parts, among them P901 677006144621, P902 677006144621, U901 TJA1040T

Commit message: Updates im Zuge des Tutorials
Parts:
- P901, P902: footprint eagle-InputOutputIO:677006144621 -> zeilhofer:Firewire-Female-WE677006144621; symbol CONN_01X06 -> CONN_01X09; InternalName (none) -> tbd
Connections:
- net GND: now also P901.7 (P7), P901.8 (P8), P901.9 (P9), P902.7 (P7), P902.8 (P8), P902.9 (P9)
Changed lines of the file:
@@
 	4200 4150 4200 4200
 $Comp
-L GND #PWR0152
+L GND #PWR0153
 U 1 1 54F00676
 P 4200 4800
-F 0 "#PWR0152" H 4200 4550 60  0001 C CNN
+F 0 "#PWR0153" H 4200 4550 60  0001 C CNN
 F 1 "GND" H 4200 4650 60  0000 C CNN
 F 2 "" H 4200 4800 60  0000 C CNN
@@
 	4200 4800 4200 4700
 $Comp
-L GND #PWR0153
+L GND #PWR0154
 U 1 1 54F006A8
 P 4800 4800
-F 0 "#PWR0153" H 4800 4550 60  0001 C CNN
+F 0 "#PWR0154" H 4800 4550 60  0001 C CNN
 F 1 "GND" H 4800 4650 60  0000 C CNN
 F 2 "" H 4800 4800 60  0000 C CNN
@@
 $EndComp
 $Comp
-L GND #PWR0154
+L GND #PWR0155
 U 1 1 54F007D4
 P 3550 4800
-F 0 "#PWR0154" H 3550 4550 60  0001 C CNN
+F 0 "#PWR0155" H 3550 4550 60  0001 C CNN
 F 1 "GND" H 3550 4650 60  0000 C CNN
 F 2 "" H 3550 4800 60  0000 C CNN
@@
 Connection ~ 6400 4250
 $Comp
-L CONN_01X06 P901
+L CONN_01X09 P901
 U 1 1 54F0145D
-P 9750 3450
-F 0 "P901" H 9750 3800 50  0000 C CNN
-F 1 "677006144621" V 9850 3450 50  0000 C CNN
-F 2 "eagle-InputOutputIO:677006144621" H 9750 3450 60  0001 C CNN
-F 3 "" H 9750 3450 60  0000 C CNN
-	1    9750 3450
-	1    0    0    -1
-$EndComp
-$Comp
-L CONN_01X06 P902
+P 10250 3600
+F 0 "P901" H 10250 4100 50  0000 C CNN
+F 1 "677006144621" V 10350 3600 50  0000 C CNN
+F 2 "zeilhofer:Firewire-Female-WE677006144621" H 10250 3600 60  0001 C CNN
+F 3 "" H 10250 3600 60  0000 C CNN
+F 4 "tbd" H 10250 3600 60  0001 C CNN "InternalName"
+	1    10250 3600
+	1    0    0    -1
+$EndComp
+$Comp
+L CONN_01X09 P902
 U 1 1 54F014A4
-P 9750 4500
-F 0 "P902" H 9750 4850 50  0000 C CNN
-F 1 "677006144621" V 9850 4500 50  0000 C CNN
-F 2 "eagle-InputOutputIO:677006144621" H 9750 4500 60  0001 C CNN
-F 3 "" H 9750 4500 60  0000 C CNN
-	1    9750 4500
-	1    0    0    -1
-$EndComp
-Wire Wire Line
-	9350 3500 9350 3500
+P 10250 4650
+F 0 "P902" H 10250 5150 50  0000 C CNN
+F 1 "677006144621" V 10350 4650 50  0000 C CNN
+F 2 "zeilhofer:Firewire-Female-WE677006144621" H 10250 4650 60  0001 C CNN
+F 3 "" H 10250 4650 60  0000 C CNN
+F 4 "tbd" H 10250 4650 60  0001 C CNN "InternalName"
+	1    10250 4650
+	1    0    0    -1
+$EndComp
+Wire Wire Line
+	8800 3500 10050 3500
 Wire Wire Line
 	9350 3500 9350 4550
 Wire Wire Line
-	9350 4550 9550 4550
+	9350 4550 10050 4550
 Connection ~ 6400 3500
 Connection ~ 9350 3500
@@
 	9450 4450 9450 3400
 Wire Wire Line
-	9450 3400 9550 3400
+	9450 3400 10050 3400
 Connection ~ 9450 4450
 Wire Wire Line
-	9550 4350 9200 4350
-$Comp
-L GND #PWR0155
+	10050 4350 9200 4350
+$Comp
+L GND #PWR0156
 U 1 1 54F016F8
 P 9200 4350
-F 0 "#PWR0155" H 9200 4100 60  0001 C CNN
+F 0 "#PWR0156" H 9200 4100 60  0001 C CNN
 F 1 "GND" H 9200 4200 60  0000 C CNN
 F 2 "" H 9200 4350 60  0000 C CNN
@@
 $EndComp
 $Comp
-L GND #PWR0156
+L GND #PWR0157
 U 1 1 54F01715
 P 9150 3300
-F 0 "#PWR0156" H 9150 3050 60  0001 C CNN
+F 0 "#PWR0157" H 9150 3050 60  0001 C CNN
 F 1 "GND" H 9150 3150 60  0000 C CNN
 F 2 "" H 9150 3300 60  0000 C CNN
@@
 $EndComp
 Wire Wire Line
-	9150 3300 9550 3300
-NoConn ~ 9550 3200
-NoConn ~ 9550 3600
-NoConn ~ 9550 3700
-NoConn ~ 9550 4250
-NoConn ~ 9550 4650
-NoConn ~ 9550 4750
+	9150 3300 10050 3300
+NoConn ~ 10050 3200
+NoConn ~ 10050 3600
+NoConn ~ 10050 3700
+NoConn ~ 10050 4250
+NoConn ~ 10050 4650
+NoConn ~ 10050 4750
 Text Notes 9300 2900 0    60   ~ 0
 Firewire Connectors\nare used for CAN
 $Comp
-L GND #PWR0157
+L GND #PWR0158
 U 1 1 54F01A23
 P 7600 4000
-F 0 "#PWR0157" H 7600 3750 60  0001 C CNN
+F 0 "#PWR0158" H 7600 3750 60  0001 C CNN
 F 1 "GND" H 7600 3850 60  0000 C CNN
 F 2 "" H 7600 4000 60  0000 C CNN
@@
 	2600 4050 2600 4200
 $Comp
-L GND #PWR0158
+L GND #PWR0159
 U 1 1 54F021C9
 P 2600 4800
-F 0 "#PWR0158" H 2600 4550 60  0001 C CNN
+F 0 "#PWR0159" H 2600 4550 60  0001 C CNN
 F 1 "GND" H 2600 4650 60  0000 C CNN
 F 2 "" H 2600 4800 60  0000 C CNN
@@
 	5350 4150 5550 4150
 Wire Wire Line
-	7150 4000 5350 4000
+	5350 4000 7150 4000
 Wire Wire Line
 	8200 3500 8200 3850
@@
 	8800 3850 8800 3500
 Wire Wire Line
-	8800 3500 9550 3500
-Wire Wire Line
-	9550 4450 8800 4450
+	8800 4450 10050 4450
 Wire Wire Line
 	8800 4450 8800 4150
+$Comp
+L GND #PWR0160
+U 1 1 55548402
+P 9750 5200
+F 0 "#PWR0160" H 9750 4950 60  0001 C CNN
+F 1 "GND" H 9750 5050 60  0000 C CNN
+F 2 "" H 9750 5200 60  0000 C CNN
+F 3 "" H 9750 5200 60  0000 C CNN
+	1    9750 5200
+	1    0    0    -1
+$EndComp
+Wire Wire Line
+	9750 4850 9750 5200
+Wire Wire Line
+	9750 5050 10050 5050
+Wire Wire Line
+	9750 4950 10050 4950
+Connection ~ 9750 5050
+Wire Wire Line
+	9750 4850 10050 4850
+Connection ~ 9750 4950
+$Comp
+L GND #PWR0161
+U 1 1 555485A9
+P 9750 4150
+F 0 "#PWR0161" H 9750 3900 60  0001 C CNN
+F 1 "GND" H 9750 4000 60  0000 C CNN
+F 2 "" H 9750 4150 60  0000 C CNN
+F 3 "" H 9750 4150 60  0000 C CNN
+	1    9750 4150
+	1    0    0    -1
+$EndComp
+Wire Wire Line
+	9750 3800 9750 4150
+Wire Wire Line
+	9750 4000 10050 4000
+Wire Wire Line
+	9750 3900 10050 3900
+Connection ~ 9750 4000
+Wire Wire Line
+	9750 3800 10050 3800
+Connection ~ 9750 3900
 $EndSCHEMATC
