File: power-meter.sch (KiCad schematic (older format))
At the start: 28 parts, among them P1101 CONN_01X02, P1102 CONN_01X02, U1101 ADL5513, U1102 REG101NA-5, X1101 SMA, X1102 SMB, X1103 SMB

Commit message: Updates im Zuge des Tutorials
Parts:
- C1105, C1107: footprint Capacitors_SMD:C_0402 -> Capacitors_SMD:C_0603
- C1110: value 47p/X7R -> 47p/C0G
